File: burn_wire_alt.kicad_sch (KiCad schematic)
At the start: 15 parts, among them J1 Conn_01x02_Pin, J2 Conn_01x02_Pin, U1 ADP2303ARDZ

Commit message: real values used for board updated schematic
Parts:
- C1: value 530u -> 330u
- C3: value 47u -> 33u
- C4: value 47u -> 22u
- R1: value 230k -> 240k
Connections:
- net Vin: no longer R5.1
- net Vout: now also R5.1
Other:
- moved on the sheet: R5
Changed lines of the file:
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@@
+	)
+	(junction
+		(at 217.17 66.04)
+		(diameter 0)
+		(color 0 0 0 0)
 	)
 	(junction
@@
 	)
 	(junction
-		(at 114.3 57.15)
-		(diameter 0)
-		(color 0 0 0 0)
-	)
-	(junction
 		(at 148.59 77.47)
 		(diameter 0)
@@
 	(wire
 		(pts
-			(xy 114.3 86.36) (xy 114.3 72.39)
+			(xy 201.93 95.25) (xy 201.93 92.71)
 		)
 		(stroke
@@
 	(wire
 		(pts
+			(xy 201.93 92.71) (xy 217.17 92.71)
+		)
+		(stroke
+			(width 0)
+			(type default)
+		)
+	)
+	(wire
+		(pts
+			(xy 217.17 66.04) (xy 217.17 85.09)
+		)
+		(stroke
+			(width 0)
+			(type default)
+		)
+	)
+	(wire
+		(pts
 			(xy 104.14 68.58) (xy 104.14 66.04)
 		)
@@
 	(wire
 		(pts
+			(xy 134.62 91.44) (xy 135.89 91.44)
+		)
+		(stroke
+			(width 0)
+			(type default)
+		)
+	)
+	(wire
+		(pts
 			(xy 161.29 60.96) (xy 162.56 60.96)
 		)
@@
 	(wire
 		(pts
-			(xy 110.49 57.15) (xy 114.3 57.15)
-		)
-		(stroke
-			(width 0)
-			(type default)
-		)
-	)
-	(wire
-		(pts
 			(xy 194.31 66.04) (xy 194.31 68.58)
 		)
@@
 	(wire
 		(pts
-			(xy 114.3 57.15) (xy 120.65 57.15)
+			(xy 110.49 57.15) (xy 120.65 57.15)
 		)
 		(stroke
@@
 	(wire
 		(pts
+			(xy 217.17 66.04) (xy 224.79 66.04)
+		)
+		(stroke
+			(width 0)
+			(type default)
+		)
+	)
+	(wire
+		(pts
 			(xy 180.34 66.04) (xy 184.15 66.04)
 		)
@@
 	(wire
 		(pts
-			(xy 135.89 71.12) (xy 135.89 86.36)
+			(xy 134.62 91.44) (xy 134.62 95.25)
 		)
 		(stroke
@@
 	(wire
 		(pts
-			(xy 114.3 57.15) (xy 114.3 64.77)
-		)
-		(stroke
-			(width 0)
-			(type default)
-		)
-	)
-	(wire
-		(pts
 			(xy 194.31 66.04) (xy 207.01 66.04)
 		)
@@
 	(wire
 		(pts
-			(xy 114.3 86.36) (xy 135.89 86.36)
+			(xy 201.93 95.25) (xy 134.62 95.25)
 		)
 		(stroke
@@
 	(wire
 		(pts
+			(xy 135.89 91.44) (xy 135.89 71.12)
+		)
+		(stroke
+			(width 0)
+			(type default)
+		)
+	)
+	(wire
+		(pts
 			(xy 167.64 66.04) (xy 172.72 66.04)
 		)
@@
 	(wire
 		(pts
-			(xy 207.01 66.04) (xy 224.79 66.04)
+			(xy 207.01 66.04) (xy 217.17 66.04)
 		)
 		(stroke
@@
 			)
 		)
-		(property "Value" "530u"
+		(property "Value" "330u"
 			(at 106.68 63.5062 0)
 			(show_name no)
@@
 			)
 		)
-		(property "Value" "47u"
+		(property "Value" "22u"
 			(at 207.772 73.152 0)
 			(show_name no)
@@
 	(symbol
 		(lib_id "Device:R_US")
-		(at 114.3 68.58 0)
+		(at 217.17 88.9 0)
 		(unit 1)
 		(body_style 1)
@@
 		(fields_autoplaced yes)
 		(property "Reference" "R5"
-			(at 116.84 67.3099 0)
+			(at 219.71 87.6299 0)
 			(show_name no)
 			(do_not_autoplace no)
@@
 		)
 		(property "Value" "100k"
-			(at 116.84 69.8499 0)
+			(at 219.71 90.1699 0)
 			(show_name no)
 			(do_not_autoplace no)
@@
 		)
 		(property "Footprint" "Resistor_SMD:R_0603_1608Metric"
-			(at 115.316 68.834 90)
+			(at 218.186 89.154 90)
 			(hide yes)
 			(show_name no)
@@
 		)
 		(property "Datasheet" ""
-			(at 114.3 68.58 0)
+			(at 217.17 88.9 0)
 			(hide yes)
 			(show_name no)
@@
 		)
 		(property "Description" "Resistor, US symbol"
-			(at 114.3 68.58 0)
+			(at 217.17 88.9 0)
 			(hide yes)
 			(show_name no)
@@
 			)
 		)
-		(property "Value" "230k"
+		(property "Value" "240k"
 			(at 123.19 63.4999 0)
 			(show_name no)
@@
 			)
 		)
-		(property "Value" "47u"
+		(property "Value" "33u"
 			(at 197.104 73.152 0)
 			(show_name no)
