File: burn_wire_alt.kicad_sch (KiCad schematic)
At the start: 15 parts, among them J1 Conn_01x02_Pin, J2 Conn_01x02_Pin, U1 ADP2303ARDZ

Commit message: applied .gitignore
Parts:
- C3: value 33u -> 22u
- C4: value 22u -> 33u
Changed lines of the file:
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@@
 			)
 		)
-		(property "Value" "22u"
+		(property "Value" "33u"
 			(at 207.772 73.152 0)
 			(show_name no)
@@
 			)
 		)
-		(property "Value" "33u"
+		(property "Value" "22u"
 			(at 197.104 73.152 0)
 			(show_name no)

Commit message: new
Parts:
- added TP1: TestPoint, Connector_PinSocket_2.54mm:PinSocket_1x01_P2.54mm_Vertical, symbol Connector:TestPoint
- R4: value 10k -> .5; footprint Resistor_SMD:R_0603_1608Metric -> Resistor_SMD:R_2512_6332Metric
Connections:
- net FB: now also R3.1; no longer R3.2, R4.1
- net Vout: no longer R3.1
- new net: R3.2, R4.1, TP1.1
Other:
- moved on the sheet: D1
